File: pcb/fs7-button.kicad_pcb (KiCad board)
At the start: 2 copper layers, 24 x 50 mm, 30 parts, among them CN1 PJ-210 3P, CN2 PJ-210 3P, J1 Conn_01x03, J4 Conn_01x06, SW1 SW_SPST, SW2 SW_Push, SW3 SW_Push, SW4 SW_Push, U1 CH32V003FxPx, U2 LP5907MFX-3.3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

Commit message: idk
Signed-off-by: 3nt3 <gott@3nt3.de>
Parts:
- removed J4: Conn_01x06, Connector_PinHeader_2.54mm:PinHeader_2x03_P2.54mm_Vertical
- added 3V3: TestPoint, TestPoint:TestPoint_Pad_D1.5mm, B.Cu at (177.3, 74.9)
- added GND: TestPoint, TestPoint:TestPoint_Pad_D1.5mm, B.Cu at (177.2, 72.0)
- added TP2: TestPoint, TestPoint:TestPoint_Pad_D1.5mm, B.Cu at (166.1, 61.8)
- added TP3: TestPoint, TestPoint:TestPoint_Pad_D1.5mm, B.Cu at (169.2, 62.0)
- added TP4: TestPoint, TestPoint:TestPoint_Pad_D1.5mm, B.Cu at (172.1, 62.2)
- added TP5: TestPoint, TestPoint:TestPoint_Pad_D1.5mm, B.Cu at (165.1, 69.0)
- SW2, SW3, SW4: footprint easyeda2kicad:KEY-SMD_4P-L6.2-W6.5-P4.50-LS8.0_SKHMXX -> easyeda2kicad:SW-SMD_4P-L5.1-W5.1-P3.70-LS6.5-TL_H1.5
- moved R3 23.4 mm to (184.5, 61.0), turned to 90 degrees
- moved D3 22.5 mm to (184.5, 64.4), turned to 90 degrees
- moved R1 21.6 mm to (163.5, 60.9), turned to 90 degrees
- moved D1 17.1 mm to (163.5, 64.3), turned to 90 degrees
- moved J1 3.61 mm to (182.0, 81.0), turned to -90 degrees
- moved U1 2.60 mm to (169.3, 62.0)
- moved C6 2.39 mm to (168.7, 76.6)
- moved U2 2.39 mm to (168.9, 79.7)
- moved C5 2.39 mm to (168.8, 83.0)
- moved C1 1.39 mm to (165.8, 56.3)
- moved C3 0.73 mm to (169.2, 51.4)
- moved C2 0.70 mm to (172.1, 54.5)
- moved Y1 0.70 mm to (169.3, 54.5)
- moved D2 0.65 mm to (163.7, 79.5)
- moved R2 0.65 mm to (163.7, 83.3)
Connections:
- CN2 pad 2: Net-(U1-PD0) -> Net-(U1-PC2)
- U1 pad 10: Net-(SW1-B) -> unconnected-(U1-PC0-Pad10)
- U1 pad 12: LED1 -> Net-(U1-PC2)
- U1 pad 2: unconnected-(U1-PD5-Pad2) -> Net-(SW1-B)
- U1 pad 8: Net-(U1-PD0) -> LED1
Routing:
- net Net-(U1-PD0): track 36.6 -> 0.00 mm, vias 2 -> 0
- net Net-(U1-PC2): track 0.00 -> 24.7 mm
- net LED2: track 26.3 -> 8.01 mm, vias 2 -> 0
- net Net-(J1-Pin_2): track 32.5 -> 19.6 mm, vias 2 -> 0
- net LED1: track 30.5 -> 18.5 mm, vias 2 -> 0
- net Net-(SW1-B): track 22.8 -> 13.9 mm
- net PC5: track 9.55 -> 2.98 mm, vias 0 -> 1
- net SW2: track 16.5 -> 10.2 mm, vias 2 -> 0
- net GND: track 37.0 -> 32.1 mm, vias 8 -> 12
- net +3V3: track 47.2 -> 44.4 mm, vias 3 -> 4
- net PC6: track 6.74 -> 4.04 mm, vias 0 -> 1
- net PC7: track 10.1 -> 7.39 mm, vias 0 -> 1
- net SW1: track 16.5 -> 13.9 mm, vias 2 -> 0
- net PC4: track 6.30 -> 4.15 mm, vias 0 -> 1
- net SW3: track 14.8 -> 12.7 mm
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Other:
- outline, holes or cut-outs redrawn

Commit message: idk
Signed-off-by: 3nt3 <gott@3nt3.de>
Parts:
- H1, H2, H3, H4: footprint MountingHole:MountingHole_2.2mm_M2_ISO14580_Pad -> MountingHole:MountingHole_2.2mm_M2_Pad_Via
Routing:
- net SW1: track 13.9 -> 19.9 mm
- net GND: track 32.1 -> 36.3 mm, vias 12 -> 15
- net SW3: track 12.7 -> 15.6 mm
- net SW2: track 10.2 -> 13.0 mm
Other:
- board text added: "FS7 HANDLE EMULATOR 3nt3 — 2025/08 — v0.2"
- board text added: "IN"
- board text added: "OUT"

Commit message: idk
Signed-off-by: 3nt3 <gott@3nt3.de>
Parts:
- added C10: 100n, Capacitor_SMD:C_0603_1608Metric_Pad1.08x0.95mm_HandSolder, F.Cu at (165.8, 52.3)
- renumbered 3V3 to TP1, GND to TP6
Connections:
- U1 pad 4: unconnected-(U1-PD7-Pad4) -> Net-(U1-PD7)
Routing:
- net Net-(U1-PD7): track 0.00 -> 17.1 mm
- net GND: track 36.3 -> 41.5 mm, vias 15 -> 17
