File: pcb/fs7-button.kicad_sch (KiCad schematic)
At the start: 24 parts, among them J1 Conn_01x03_Socket, J2 AudioJack3, J3 Conn_01x06, J4 Conn_01x06, SW1 SW_SPST, U1 CH32V003FxPx, U2 LP5907MFX-3.3, Y1 Crystal_GND24

Commit message: some kind of version
Signed-off-by: 3nt3 <gott@3nt3.de>
Parts:
- removed J1: Conn_01x03_Socket, symbol Connector:Conn_01x03_Socket
- removed J2: AudioJack3, symbol Connector_Audio:AudioJack3
- removed J3: Conn_01x06, symbol Connector_Generic:Conn_01x06
- added C7, C8, C9: 100n, Capacitor_SMD:C_0603_1608Metric_Pad1.08x0.95mm_HandSolder, symbol Device:C
- added CN1, CN2: PJ-210 3P, easyeda2kicad:AUDIO-TH_PJ-210-3P, symbol easyeda2kicad:PJ-2103P
- added J1: Conn_01x03, Connector_PinHeader_2.54mm:PinHeader_1x03_P2.54mm_Vertical, symbol Connector_Generic:Conn_01x03
- added SW2, SW3, SW4: SW_Push, easyeda2kicad:SW-SMD_4P-L5.1-W5.1-P3.70-LS6.5-TL_H1.5, symbol Switch:SW_Push
- C1, C4, C5, C6: footprint (none) -> Capacitor_SMD:C_0603_1608Metric_Pad1.08x0.95mm_HandSolder
- C2, C3: value 1u -> 14p; footprint (none) -> Capacitor_SMD:C_0603_1608Metric_Pad1.08x0.95mm_HandSolder
- D1, D2, D3: footprint (none) -> LED_SMD:LED_0603_1608Metric_Pad1.05x0.95mm_HandSolder
- H1, H2, H3, H4: footprint (none) -> MountingHole:MountingHole_2.2mm_M2_ISO14580_Pad
- J4: footprint (none) -> Connector_PinHeader_2.54mm:PinHeader_2x03_P2.54mm_Vertical
- R1, R3: footprint (none) -> Resistor_SMD:R_0603_1608Metric_Pad0.98x0.95mm_HandSolder
- R2: value 1u -> 680R; footprint (none) -> Resistor_SMD:R_0603_1608Metric_Pad0.98x0.95mm_HandSolder
- SW1: footprint (none) -> easyeda2kicad:SW-TH_SK12D07VG5-1
- Y1: footprint (none) -> Crystal:Crystal_SMD_3225-4Pin_3.2x2.5mm
Connections:
- net +3V3: now also J4.6 (Pin_6), J1.3 (Pin_3); no longer J4.1 (Pin_1)
- net GND: now also J4.1 (Pin_1), C7.2, C8.2, C9.2, CN1.1, CN2.1, J1.1 (Pin_1), SW2.2, SW3.2, SW4.2; no longer J4.6 (Pin_6)
- net LED1: no longer R1.2
- net LED2: now also R1.2
- net PC4: now also J4.5 (Pin_5); no longer J4.2 (Pin_2)
- net PC5: now also J4.4 (Pin_4); no longer J4.3 (Pin_3)
- net PC6: now also J4.3 (Pin_3); no longer J4.4 (Pin_4)
- net PC7: now also J4.2 (Pin_2); no longer J4.5 (Pin_5)
- net SW1: now also C7.1, SW3.1
- net SW2: now also C8.1, SW4.1
- net SW3: now also C9.1, SW2.1
- net VBUS: now also CN1.3, CN2.3
- net at U1.11 (PC1): now also CN1.2
- net at U1.18 (PD1): now also J1.2 (Pin_2)
- net at U1.8 (PD0): now also CN2.2
- net PD5: no longer names the net of U1.2 (PD5)
- net PD6: no longer names the net of U1.3 (PD6)
- net PD7: no longer names the net of U1.4 (PD7)
- no-connect marks 0 -> 3
Other:
- note added: "Push buttons"
- moved on the sheet: D1, D3, J4, R1, R3

Commit message: idk
Signed-off-by: 3nt3 <gott@3nt3.de>
Parts:
- removed J4: Conn_01x06, Connector_PinHeader_2.54mm:PinHeader_2x03_P2.54mm_Vertical, symbol Connector_Generic:Conn_01x06
- added TP1, TP2, TP3, TP4, TP5, TP6: TestPoint, TestPoint:TestPoint_Pad_D1.5mm, symbol Connector:TestPoint
Connections:
- net +3V3: now also TP1.1
- net GND: now also TP6.1
- net LED1: now also U1.8 (PD0); no longer U1.12 (PC2)
- net PC4: now also TP2.1
- net PC5: now also TP3.1
- net PC6: now also TP4.1
- net PC7: now also TP5.1
- net at CN2.2: now also U1.12 (PC2); no longer U1.8 (PD0)
- net at C4.2, SW1.2 (B): now also U1.2 (PD5); no longer U1.10 (PC0)
- no-connect marks 3 -> 2
Other:
- moved on the sheet: C4, C7, C8, C9, CN1, CN2, SW1, SW2, SW3, SW4

Commit message: idk
Signed-off-by: 3nt3 <gott@3nt3.de>
Parts:
- H1, H2, H3, H4: footprint MountingHole:MountingHole_2.2mm_M2_ISO14580_Pad -> MountingHole:MountingHole_2.2mm_M2_Pad_Via
Changed lines of the file:
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@@
 			)
 		)
-		(property "Footprint" "MountingHole:MountingHole_2.2mm_M2_ISO14580_Pad"
+		(property "Footprint" "MountingHole:MountingHole_2.2mm_M2_Pad_Via"
 			(at 146.05 142.24 0)
 			(effects
@@
 			)
 		)
-		(property "Footprint" "MountingHole:MountingHole_2.2mm_M2_ISO14580_Pad"
+		(property "Footprint" "MountingHole:MountingHole_2.2mm_M2_Pad_Via"
 			(at 135.89 142.24 0)
 			(effects
@@
 			)
 		)
-		(property "Footprint" "MountingHole:MountingHole_2.2mm_M2_ISO14580_Pad"
+		(property "Footprint" "MountingHole:MountingHole_2.2mm_M2_Pad_Via"
 			(at 151.13 142.24 0)
 			(effects
@@
 			)
 		)
-		(property "Footprint" "MountingHole:MountingHole_2.2mm_M2_ISO14580_Pad"
+		(property "Footprint" "MountingHole:MountingHole_2.2mm_M2_Pad_Via"
 			(at 140.97 142.24 0)
 			(effects

Commit message: idk
Signed-off-by: 3nt3 <gott@3nt3.de>
Parts:
- added C10: 100n, Capacitor_SMD:C_0603_1608Metric_Pad1.08x0.95mm_HandSolder, symbol Device:C
Connections:
- net GND: now also C10.2
- net at U1.4 (PD7): now also C10.1
- no-connect marks 2 -> 1
Changed lines of the file:
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@@
 		(at 154.94 97.79)
 	)
-	(no_connect
-		(at 154.94 100.33)
-	)
 	(wire
 		(pts
@@
 	(wire
 		(pts
+			(xy 161.29 100.33) (xy 161.29 109.22)
+		)
+		(stroke
+			(width 0)
+			(type default)
+		)
+	)
+	(wire
+		(pts
 			(xy 223.52 123.19) (xy 218.44 123.19)
 		)
@@
 		(pts
 			(xy 250.19 127) (xy 250.19 123.19)
+		)
+		(stroke
+			(width 0)
+			(type default)
+		)
+	)
+	(wire
+		(pts
+			(xy 154.94 100.33) (xy 161.29 100.33)
 		)
 		(stroke
@@
 	(symbol
 		(lib_id "Device:C")
+		(at 161.29 113.03 0)
+		(unit 1)
+		(exclude_from_sim no)
+		(in_bom yes)
+		(on_board yes)
+		(dnp no)
+		(fields_autoplaced yes)
+		(property "Reference" "C10"
+			(at 165.1 111.7599 0)
+			(effects
+				(font
+					(size 1.27 1.27)
+				)
+				(justify left)
+			)
+		)
+		(property "Value" "100n"
+			(at 165.1 114.2999 0)
+			(effects
+				(font
+					(size 1.27 1.27)
+				)
+				(justify left)
+			)
+		)
+		(property "Footprint" "Capacitor_SMD:C_0603_1608Metric_Pad1.08x0.95mm_HandSolder"
+			(at 162.2552 116.84 0)
+			(effects
+				(font
+					(size 1.27 1.27)
+				)
+				(hide yes)
+			)
+		)
+		(property "Datasheet" "~"
+			(at 161.29 113.03 0)
+			(effects
+				(font
+					(size 1.27 1.27)
+				)
+				(hide yes)
+			)
+		)
+		(property "Description" "Unpolarized capacitor"
+			(at 161.29 113.03 0)
+			(effects
+				(font
+					(size 1.27 1.27)
+				)
+				(hide yes)
+			)
+		)
+		(pin "2"
+		)
+		(pin "1"
+		)
+		(instances
+			(project ""
+				(path "/f5fe6669-9eae-4313-a9e4-62cdbf04e572"
+					(reference "C10")
+					(unit 1)
+				)
+			)
+		)
+	)
+	(symbol
+		(lib_id "Device:C")
 		(at 213.36 127 90)
 		(unit 1)
@@
 					(unit 1)
 				)
+			)
+		)
+	)
+	(symbol
+		(lib_id "power:GND")
+		(at 161.29 116.84 0)
+		(unit 1)
+		(exclude_from_sim no)
+		(in_bom yes)
+		(on_board yes)
+		(dnp no)
+		(fields_autoplaced yes)
+		(property "Reference" "#PWR023"
+			(at 161.29 123.19 0)
+			(effects
+				(font
+					(size 1.27 1.27)
+				)
+				(hide yes)
+			)
+		)
+		(property "Value" "GND"
+			(at 161.29 121.92 0)
+			(effects
+				(font
+					(size 1.27 1.27)
+				)
+			)
+		)
+		(property "Footprint" ""
+			(at 161.29 116.84 0)
+			(effects
+				(font
+					(size 1.27 1.27)
+				)
+				(hide yes)
+			)
+		)
+		(property "Datasheet" ""
+			(at 161.29 116.84 0)
+			(effects
+				(font
+					(size 1.27 1.27)
+				)
+				(hide yes)
+			)
+		)
+		(property "Description" "Power symbol creates a global label with name \"GND\" , ground"
+			(at 161.29 116.84 0)
+			(effects
+				(font
+					(size 1.27 1.27)
+				)
+				(hide yes)
+			)
+		)
+		(pin "1"
+		)
+		(instances
+			(project ""
+				(path "/f5fe6669-9eae-4313-a9e4-62cdbf04e572"
+					(reference "#PWR023")
+					(unit 1)
+				)
